File: kicad/pc/v0.2/MiniPC.kicad_pcb (KiCad board)
At the start: 2 copper layers, 145.7 x 82.2 mm, 83 parts, among them J1 Conn_02x06_Odd_Even, J2 HDMI_A, J3 Programmer, J4 SD_Card, J5 Cassette Output, J6 Mini-DIN-6, J7 USB_C_Receptacle_PowerOnly_6P, J8 Probe, SW1 ESP_RESET, SW2 STATUS, SW3 SW_DIP_x04, SW4 PC_RESET, U1 APS6404L-3SQRx-SN, U2 ESP32-WROVER-B

Commit message: Version 0.2 (April) of MiniPC PCB
Parts:
- removed the C12 at (140.1, 124.0)
- removed G*** (x2): LOGO, LOGO
- removed the R10 at (129.4, 124.0)
- removed the R11 at (127.3, 124.0)
- removed the R12 at (125.2, 124.0)
- removed the R13 at (123.2, 124.0)
- removed the R6 at (137.7, 124.0)
- removed the R7 at (135.7, 124.0)
- removed the R8 at (133.6, 124.0)
- removed the R9 at (131.5, 124.0)
- moved R21 115.1 mm to (181.7, 130.4), turned to -90 degrees
- moved SW3 97.5 mm to (166.8, 139.8), turned to 180 degrees
- moved C2 20.8 mm to (146.1, 98.1), turned to -90 degrees
- moved C3 17.7 mm to (143.8, 98.1), turned to -90 degrees
- moved U1 11.2 mm to (138.8, 98.9), turned to 0 degrees
- moved R1 10.1 mm to (133.8, 99.5)
- moved SW2 4.27 mm to (178.7, 139.8)
- moved SW1 3.20 mm to (190.6, 139.8)
- renumbered C13 to C12, C14 to C13, C15 to C14, C16 to C15, C17 to C16, C18 to C17, C19 to C18, D6 to D5, D5 to D6, J8 to J4, J4 to J5, J5 to J6, J6 to J7, J7 to J8, R18 to R10, R19 to R11, R20 to R12, R21 to R13, R22 to R14, R23 to R15, R24 to R16, R25 to R17, R26 to R18, R27 to R19, R28 to R20, R37 to R21, R29 to R22, R30 to R23, R31 to R24, R32 to R25, R33 to R26, R34 to R27, R35 to R28, R36 to R29, R14 to R6, R15 to R7, R16 to R8, R17 to R9, SW4 to SW3, SW3 to SW4
Connections:
- Conn1 pad 15: unconnected-(Conn1A-T10-Pad15) -> CS_SD
- Conn1 pad 28: unconnected-(Conn1A-R16-Pad28) -> PS2_CLK
- Conn1 pad 30: unconnected-(Conn1A-P15-Pad30) -> PS2_DATA
- Conn1 pad 42: PSRAM_CE_n -> PSRAM_SIO2
- Conn1 pad 46: PSRAM_SIO2 -> PSRAM_CE_n
Routing:
- net PC_RESET: track 59.6 -> 152.3 mm, vias 0 -> 2
- net +3V3: track 539.4 -> 457.6 mm, vias 17 -> 9
- net CS_SD: track 28.3 -> 96.3 mm, vias 2 -> 4
- net PS2_CLK: track 88.4 -> 134.6 mm
- net PS2_DATA: track 94.8 -> 139.5 mm
- net PSRAM_CE_n: track 22.2 -> 8.63 mm
- net PSRAM_SIO3: track 20.5 -> 7.61 mm
- net PSRAM_SCLK: track 21.3 -> 9.61 mm
- net PSRAM_SIO0: track 21.9 -> 11.2 mm
- net PSRAM_SIO1: track 15.5 -> 7.88 mm
- net PSRAM_SIO2: track 16.2 -> 9.62 mm
- net GND: track 346.9 -> 349.9 mm, vias 74 -> 80
- net ESP_RESET: track 76.9 -> 78.0 mm
- net /D1+: track 16.8 -> 15.9 mm
- net ID0: track 52.1 -> 51.2 mm
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Other:
- board text added: "MiniPC V0.2 April 2026"
- board text added: "Sound"
- board text removed: "3V3"
- board text removed: "MiniPC V0.2 March 2026"
- board text removed: "Output"
