File: kicad/pc/v0.2/MiniPC.kicad_sch (KiCad schematic)
At the start: 81 parts, among them J1 Conn_02x06_Odd_Even, J2 HDMI_A, J3 Programmer, J4 SD_Card, J5 Cassette Output, J6 Mini-DIN-6, J7 USB_C_Receptacle_PowerOnly_6P, J8 Probe, SW1 ESP_RESET, SW2 STATUS, SW3 SW_DIP_x04, SW4 PC_RESET, U1 APS6404L-3SQRx-SN, U2 ESP32-WROVER-B

Commit message: Version 0.2 (April) of MiniPC PCB
Parts:
- removed C12: 100n, Capacitor_SMD:C_0805_2012Metric_Pad1.18x1.45mm_HandSolder, symbol Device:C
- removed R10, R11, R12, R13, R6, R7, R8, R9: 50, Resistor_SMD:R_0805_2012Metric_Pad1.20x1.40mm_HandSolder, symbol Device:R
- U2: LCSC C967023 -> C529589
- renumbered C13 to C12, C14 to C13, C15 to C14, C16 to C15, C17 to C16, C18 to C17, C19 to C18, D6 to D5, D5 to D6, J8 to J4, J4 to J5, J5 to J6, J6 to J7, J7 to J8, R18 to R10, R19 to R11, R20 to R12, R21 to R13, R22 to R14, R23 to R15, R24 to R16, R25 to R17, R26 to R18, R27 to R19, R28 to R20, R37 to R21, R29 to R22, R30 to R23, R31 to R24, R32 to R25, R33 to R26, R34 to R27, R35 to R28, R36 to R29, R14 to R6, R15 to R7, R16 to R8, R17 to R9, SW4 to SW3, SW3 to SW4
Connections:
- net CS_SD: now also Conn1.15 (T10)
- net PS2_CLK: now also Conn1.28 (R16)
- net PS2_DATA: now also Conn1.30 (P15)
- net PSRAM_CE_n: now also Conn1.46 (L14); no longer Conn1.42 (N14)
- net PSRAM_SIO2: now also Conn1.42 (N14); no longer Conn1.46 (L14)
- no-connect marks 61 -> 58
